Commit message: Replace '__' prefixes (#579) (e-Series)

File: ur_description/urdf/ur3.urdf.xacro (robot description, xacro)
@@ -26,5 +26,5 @@
     safety_k_position:=20
     kinematics_file">
-    <xacro:property name="__kinematics" value="${kinematics_file['kinematics']}"/>
+    <xacro:property name="config_kinematics" value="${kinematics_file['kinematics']}"/>
     <!-- Inertia parameters -->
     <xacro:property name="base_mass" value="2.0" />  <!-- This mass might be incorrect -->
@@ -74,5 +74,5 @@
       <parent link="${prefix}base_link" />
       <child link = "${prefix}shoulder_link" />
-      <origin xyz="${__kinematics['shoulder']['x']} ${__kinematics['shoulder']['y']} ${__kinematics['shoulder']['z']}" rpy="${__kinematics['shoulder']['roll']} ${__kinematics['shoulder']['pitch']} ${__kinematics['shoulder']['yaw'] + base_correction}" />
+      <origin xyz="${config_kinematics['shoulder']['x']} ${config_kinematics['shoulder']['y']} ${config_kinematics['shoulder']['z']}" rpy="${config_kinematics['shoulder']['roll']} ${config_kinematics['shoulder']['pitch']} ${config_kinematics['shoulder']['yaw'] + base_correction}" />
       <axis xyz="0 0 1" />
       <xacro:unless value="${joint_limited}">
@@ -113,5 +113,5 @@
       <parent link="${prefix}shoulder_link" />
       <child link = "${prefix}upper_arm_link" />
-      <origin xyz="${__kinematics['upper_arm']['x']} ${__kinematics['upper_arm']['y']} ${__kinematics['upper_arm']['z']}" rpy="${__kinematics['upper_arm']['roll']} ${__kinematics['upper_arm']['pitch']} ${__kinematics['upper_arm']['yaw']}" />
+      <origin xyz="${config_kinematics['upper_arm']['x']} ${config_kinematics['upper_arm']['y']} ${config_kinematics['upper_arm']['z']}" rpy="${config_kinematics['upper_arm']['roll']} ${config_kinematics['upper_arm']['pitch']} ${config_kinematics['upper_arm']['yaw']}" />
       <axis xyz="0 0 1" />
       <xacro:unless value="${joint_limited}">
@@ -145,6 +145,6 @@
         </geometry>
       </collision>
-      <xacro:cylinder_inertial radius="0.075" length="${-1*__kinematics['forearm']['x']}" mass="${upper_arm_mass}">
-        <origin xyz="${0.5*__kinematics['forearm']['x']} 0.0 ${upper_arm_inertia_offset}" rpy="0 ${pi/2} 0" />
+      <xacro:cylinder_inertial radius="0.075" length="${-1*config_kinematics['forearm']['x']}" mass="${upper_arm_mass}">
+        <origin xyz="${0.5*config_kinematics['forearm']['x']} 0.0 ${upper_arm_inertia_offset}" rpy="0 ${pi/2} 0" />
       </xacro:cylinder_inertial>
     </link>
@@ -152,5 +152,5 @@
       <parent link="${prefix}upper_arm_link" />
       <child link = "${prefix}forearm_link" />
-      <origin xyz="${__kinematics['forearm']['x']} ${__kinematics['forearm']['y']} ${__kinematics['forearm']['z']}" rpy="${__kinematics['forearm']['roll']} ${__kinematics['forearm']['pitch']} ${__kinematics['forearm']['yaw']}" />
+      <origin xyz="${config_kinematics['forearm']['x']} ${config_kinematics['forearm']['y']} ${config_kinematics['forearm']['z']}" rpy="${config_kinematics['forearm']['roll']} ${config_kinematics['forearm']['pitch']} ${config_kinematics['forearm']['yaw']}" />
       <axis xyz="0 0 1" />
       <xacro:unless value="${joint_limited}">
@@ -184,6 +184,6 @@
         </geometry>
       </collision>
-      <xacro:cylinder_inertial radius="0.075" length="${-1*__kinematics['wrist_1']['x']}" mass="${forearm_mass}">
-        <origin xyz="${0.5*__kinematics['forearm']['x']} 0.0 ${elbow_offset}" rpy="0 ${pi/2} 0" />
+      <xacro:cylinder_inertial radius="0.075" length="${-1*config_kinematics['wrist_1']['x']}" mass="${forearm_mass}">
+        <origin xyz="${0.5*config_kinematics['forearm']['x']} 0.0 ${elbow_offset}" rpy="0 ${pi/2} 0" />
       </xacro:cylinder_inertial>
     </link>
@@ -191,5 +191,5 @@
       <parent link="${prefix}forearm_link" />
       <child link = "${prefix}wrist_1_link" />
-      <origin xyz="${__kinematics['wrist_1']['x']} ${__kinematics['wrist_1']['y']} ${__kinematics['wrist_1']['z']}" rpy="${__kinematics['wrist_1']['roll']} ${__kinematics['wrist_1']['pitch']} ${__kinematics['wrist_1']['yaw']}" />
+      <origin xyz="${config_kinematics['wrist_1']['x']} ${config_kinematics['wrist_1']['y']} ${config_kinematics['wrist_1']['z']}" rpy="${config_kinematics['wrist_1']['roll']} ${config_kinematics['wrist_1']['pitch']} ${config_kinematics['wrist_1']['yaw']}" />
       <axis xyz="0 0 1" />
       <xacro:unless value="${joint_limited}">
@@ -223,5 +223,5 @@
         </geometry>
       </collision>
-      <xacro:cylinder_inertial radius="0.075" length="${-1*__kinematics['wrist_2']['y']}" mass="${wrist_1_mass}">
+      <xacro:cylinder_inertial radius="0.075" length="${-1*config_kinematics['wrist_2']['y']}" mass="${wrist_1_mass}">
         <origin xyz="0.0 0.0 0.0" rpy="0 0 0" />
       </xacro:cylinder_inertial>
@@ -230,5 +230,5 @@
       <parent link="${prefix}wrist_1_link" />
       <child link = "${prefix}wrist_2_link" />
-      <origin xyz="${__kinematics['wrist_2']['x']} ${__kinematics['wrist_2']['y']} ${__kinematics['wrist_2']['z']}" rpy="${__kinematics['wrist_2']['roll']} ${__kinematics['wrist_2']['pitch']} ${__kinematics['wrist_2']['yaw']}" />
+      <origin xyz="${config_kinematics['wrist_2']['x']} ${config_kinematics['wrist_2']['y']} ${config_kinematics['wrist_2']['z']}" rpy="${config_kinematics['wrist_2']['roll']} ${config_kinematics['wrist_2']['pitch']} ${config_kinematics['wrist_2']['yaw']}" />
       <axis xyz="0 0 1" />
       <xacro:unless value="${joint_limited}">
@@ -262,5 +262,5 @@
         </geometry>
       </collision>
-      <xacro:cylinder_inertial radius="0.075" length="${__kinematics['wrist_3']['y']}" mass="${wrist_2_mass}">
+      <xacro:cylinder_inertial radius="0.075" length="${config_kinematics['wrist_3']['y']}" mass="${wrist_2_mass}">
         <origin xyz="0.0 0.0 0.0" rpy="0 0 0" />
       </xacro:cylinder_inertial>
@@ -269,5 +269,5 @@
       <parent link="${prefix}wrist_2_link" />
       <child link = "${prefix}wrist_3_link" />
-      <origin xyz="${__kinematics['wrist_3']['x']} ${__kinematics['wrist_3']['y']} ${__kinematics['wrist_3']['z']}" rpy="${__kinematics['wrist_3']['roll']} ${__kinematics['wrist_3']['pitch']} ${__kinematics['wrist_3']['yaw']}" />
+      <origin xyz="${config_kinematics['wrist_3']['x']} ${config_kinematics['wrist_3']['y']} ${config_kinematics['wrist_3']['z']}" rpy="${config_kinematics['wrist_3']['roll']} ${config_kinematics['wrist_3']['pitch']} ${config_kinematics['wrist_3']['yaw']}" />
       <axis xyz="0 0 1" />
       <xacro:unless value="${joint_limited}">

Commit message: Replace '__' prefixes (e-Series)

File: ur_description/urdf/ur3.urdf.xacro (robot description, xacro)
@@ -26,5 +26,5 @@
     safety_k_position:=20
     kinematics_file">
-    <xacro:property name="config_kinematicskinematics" value="${kinematics_file['kinematics']}"/>
+    <xacro:property name="config_kinematics" value="${kinematics_file['kinematics']}"/>
     <!-- Inertia parameters -->
     <xacro:property name="base_mass" value="2.0" />  <!-- This mass might be incorrect -->
@@ -74,5 +74,5 @@
       <parent link="${prefix}base_link" />
       <child link = "${prefix}shoulder_link" />
-      <origin xyz="${config_kinematicskinematics['shoulder']['x']} ${config_kinematicskinematics['shoulder']['y']} ${config_kinematicskinematics['shoulder']['z']}" rpy="${config_kinematicskinematics['shoulder']['roll']} ${config_kinematicskinematics['shoulder']['pitch']} ${config_kinematicskinematics['shoulder']['yaw'] + base_correction}" />
+      <origin xyz="${config_kinematics['shoulder']['x']} ${config_kinematics['shoulder']['y']} ${config_kinematics['shoulder']['z']}" rpy="${config_kinematics['shoulder']['roll']} ${config_kinematics['shoulder']['pitch']} ${config_kinematics['shoulder']['yaw'] + base_correction}" />
       <axis xyz="0 0 1" />
       <xacro:unless value="${joint_limited}">
@@ -113,5 +113,5 @@
       <parent link="${prefix}shoulder_link" />
       <child link = "${prefix}upper_arm_link" />
-      <origin xyz="${config_kinematicskinematics['upper_arm']['x']} ${config_kinematicskinematics['upper_arm']['y']} ${config_kinematicskinematics['upper_arm']['z']}" rpy="${config_kinematicskinematics['upper_arm']['roll']} ${config_kinematicskinematics['upper_arm']['pitch']} ${config_kinematicskinematics['upper_arm']['yaw']}" />
+      <origin xyz="${config_kinematics['upper_arm']['x']} ${config_kinematics['upper_arm']['y']} ${config_kinematics['upper_arm']['z']}" rpy="${config_kinematics['upper_arm']['roll']} ${config_kinematics['upper_arm']['pitch']} ${config_kinematics['upper_arm']['yaw']}" />
       <axis xyz="0 0 1" />
       <xacro:unless value="${joint_limited}">
@@ -145,6 +145,6 @@
         </geometry>
       </collision>
-      <xacro:cylinder_inertial radius="0.075" length="${-1*config_kinematicskinematics['forearm']['x']}" mass="${upper_arm_mass}">
-        <origin xyz="${0.5*config_kinematicskinematics['forearm']['x']} 0.0 ${upper_arm_inertia_offset}" rpy="0 ${pi/2} 0" />
+      <xacro:cylinder_inertial radius="0.075" length="${-1*config_kinematics['forearm']['x']}" mass="${upper_arm_mass}">
+        <origin xyz="${0.5*config_kinematics['forearm']['x']} 0.0 ${upper_arm_inertia_offset}" rpy="0 ${pi/2} 0" />
       </xacro:cylinder_inertial>
     </link>
@@ -152,5 +152,5 @@
       <parent link="${prefix}upper_arm_link" />
       <child link = "${prefix}forearm_link" />
-      <origin xyz="${config_kinematicskinematics['forearm']['x']} ${config_kinematicskinematics['forearm']['y']} ${config_kinematicskinematics['forearm']['z']}" rpy="${config_kinematicskinematics['forearm']['roll']} ${config_kinematicskinematics['forearm']['pitch']} ${config_kinematicskinematics['forearm']['yaw']}" />
+      <origin xyz="${config_kinematics['forearm']['x']} ${config_kinematics['forearm']['y']} ${config_kinematics['forearm']['z']}" rpy="${config_kinematics['forearm']['roll']} ${config_kinematics['forearm']['pitch']} ${config_kinematics['forearm']['yaw']}" />
       <axis xyz="0 0 1" />
       <xacro:unless value="${joint_limited}">
@@ -184,6 +184,6 @@
         </geometry>
       </collision>
-      <xacro:cylinder_inertial radius="0.075" length="${-1*config_kinematicskinematics['wrist_1']['x']}" mass="${forearm_mass}">
-        <origin xyz="${0.5*config_kinematicskinematics['forearm']['x']} 0.0 ${elbow_offset}" rpy="0 ${pi/2} 0" />
+      <xacro:cylinder_inertial radius="0.075" length="${-1*config_kinematics['wrist_1']['x']}" mass="${forearm_mass}">
+        <origin xyz="${0.5*config_kinematics['forearm']['x']} 0.0 ${elbow_offset}" rpy="0 ${pi/2} 0" />
       </xacro:cylinder_inertial>
     </link>
@@ -191,5 +191,5 @@
       <parent link="${prefix}forearm_link" />
       <child link = "${prefix}wrist_1_link" />
-      <origin xyz="${config_kinematicskinematics['wrist_1']['x']} ${config_kinematicskinematics['wrist_1']['y']} ${config_kinematicskinematics['wrist_1']['z']}" rpy="${config_kinematicskinematics['wrist_1']['roll']} ${config_kinematicskinematics['wrist_1']['pitch']} ${config_kinematicskinematics['wrist_1']['yaw']}" />
+      <origin xyz="${config_kinematics['wrist_1']['x']} ${config_kinematics['wrist_1']['y']} ${config_kinematics['wrist_1']['z']}" rpy="${config_kinematics['wrist_1']['roll']} ${config_kinematics['wrist_1']['pitch']} ${config_kinematics['wrist_1']['yaw']}" />
       <axis xyz="0 0 1" />
       <xacro:unless value="${joint_limited}">
@@ -223,5 +223,5 @@
         </geometry>
       </collision>
-      <xacro:cylinder_inertial radius="0.075" length="${-1*config_kinematicskinematics['wrist_2']['y']}" mass="${wrist_1_mass}">
+      <xacro:cylinder_inertial radius="0.075" length="${-1*config_kinematics['wrist_2']['y']}" mass="${wrist_1_mass}">
         <origin xyz="0.0 0.0 0.0" rpy="0 0 0" />
       </xacro:cylinder_inertial>
@@ -230,5 +230,5 @@
       <parent link="${prefix}wrist_1_link" />
       <child link = "${prefix}wrist_2_link" />
-      <origin xyz="${config_kinematicskinematics['wrist_2']['x']} ${config_kinematicskinematics['wrist_2']['y']} ${config_kinematicskinematics['wrist_2']['z']}" rpy="${config_kinematicskinematics['wrist_2']['roll']} ${config_kinematicskinematics['wrist_2']['pitch']} ${config_kinematicskinematics['wrist_2']['yaw']}" />
+      <origin xyz="${config_kinematics['wrist_2']['x']} ${config_kinematics['wrist_2']['y']} ${config_kinematics['wrist_2']['z']}" rpy="${config_kinematics['wrist_2']['roll']} ${config_kinematics['wrist_2']['pitch']} ${config_kinematics['wrist_2']['yaw']}" />
       <axis xyz="0 0 1" />
       <xacro:unless value="${joint_limited}">
@@ -262,5 +262,5 @@
         </geometry>
       </collision>
-      <xacro:cylinder_inertial radius="0.075" length="${config_kinematicskinematics['wrist_3']['y']}" mass="${wrist_2_mass}">
+      <xacro:cylinder_inertial radius="0.075" length="${config_kinematics['wrist_3']['y']}" mass="${wrist_2_mass}">
         <origin xyz="0.0 0.0 0.0" rpy="0 0 0" />
       </xacro:cylinder_inertial>
@@ -269,5 +269,5 @@
       <parent link="${prefix}wrist_2_link" />
       <child link = "${prefix}wrist_3_link" />
-      <origin xyz="${config_kinematicskinematics['wrist_3']['x']} ${config_kinematicskinematics['wrist_3']['y']} ${config_kinematicskinematics['wrist_3']['z']}" rpy="${config_kinematicskinematics['wrist_3']['roll']} ${config_kinematicskinematics['wrist_3']['pitch']} ${config_kinematicskinematics['wrist_3']['yaw']}" />
+      <origin xyz="${config_kinematics['wrist_3']['x']} ${config_kinematics['wrist_3']['y']} ${config_kinematics['wrist_3']['z']}" rpy="${config_kinematics['wrist_3']['roll']} ${config_kinematics['wrist_3']['pitch']} ${config_kinematics['wrist_3']['yaw']}" />
       <axis xyz="0 0 1" />
       <xacro:unless value="${joint_limited}">

File: ur_e_description/urdf/ur16e.urdf.xacro (robot description, xacro)
@@ -27,5 +27,5 @@
     safety_k_position:=20
     kinematics_file">
-    <xacro:property name="__kinematics" value="${kinematics_file['kinematics']}"/>
+    <xacro:property name="config_kinematics" value="${kinematics_file['kinematics']}"/>
     <!-- Inertia parameters -->
     <xacro:property name="base_mass" value="4.0" />  <!-- This mass might be incorrect -->
@@ -75,5 +75,5 @@
       <parent link="${prefix}base_link" />
       <child link = "${prefix}shoulder_link" />
-      <origin xyz="${__kinematics['shoulder']['x']} ${__kinematics['shoulder']['y']} ${__kinematics['shoulder']['z']}" rpy="${__kinematics['shoulder']['roll']} ${__kinematics['shoulder']['pitch']} ${__kinematics['shoulder']['yaw'] + base_correction}" />
+      <origin xyz="${config_kinematics['shoulder']['x']} ${config_kinematics['shoulder']['y']} ${config_kinematics['shoulder']['z']}" rpy="${config_kinematics['shoulder']['roll']} ${config_kinematics['shoulder']['pitch']} ${config_kinematics['shoulder']['yaw'] + base_correction}" />
       <axis xyz="0 0 1" />
       <xacro:unless value="${joint_limited}">
@@ -114,5 +114,5 @@
       <parent link="${prefix}shoulder_link" />
       <child link = "${prefix}upper_arm_link" />
-      <origin xyz="${__kinematics['upper_arm']['x']} ${__kinematics['upper_arm']['y']} ${__kinematics['upper_arm']['z']}" rpy="${__kinematics['upper_arm']['roll']} ${__kinematics['upper_arm']['pitch']} ${__kinematics['upper_arm']['yaw']}" />
+      <origin xyz="${config_kinematics['upper_arm']['x']} ${config_kinematics['upper_arm']['y']} ${config_kinematics['upper_arm']['z']}" rpy="${config_kinematics['upper_arm']['roll']} ${config_kinematics['upper_arm']['pitch']} ${config_kinematics['upper_arm']['yaw']}" />
       <axis xyz="0 0 1" />
       <xacro:unless value="${joint_limited}">
@@ -146,6 +146,6 @@
         </geometry>
       </collision>
-      <xacro:cylinder_inertial radius="0.075" length="${-1*__kinematics['forearm']['x']}" mass="${upper_arm_mass}">
-        <origin xyz="${0.5*__kinematics['forearm']['x']} 0.0 ${upper_arm_inertia_offset}" rpy="0 ${pi/2} 0" />
+      <xacro:cylinder_inertial radius="0.075" length="${-1*config_kinematics['forearm']['x']}" mass="${upper_arm_mass}">
+        <origin xyz="${0.5*config_kinematics['forearm']['x']} 0.0 ${upper_arm_inertia_offset}" rpy="0 ${pi/2} 0" />
       </xacro:cylinder_inertial>
     </link>
@@ -153,5 +153,5 @@
       <parent link="${prefix}upper_arm_link" />
       <child link = "${prefix}forearm_link" />
-      <origin xyz="${__kinematics['forearm']['x']} ${__kinematics['forearm']['y']} ${__kinematics['forearm']['z']}" rpy="${__kinematics['forearm']['roll']} ${__kinematics['forearm']['pitch']} ${__kinematics['forearm']['yaw']}" />
+      <origin xyz="${config_kinematics['forearm']['x']} ${config_kinematics['forearm']['y']} ${config_kinematics['forearm']['z']}" rpy="${config_kinematics['forearm']['roll']} ${config_kinematics['forearm']['pitch']} ${config_kinematics['forearm']['yaw']}" />
       <axis xyz="0 0 1" />
       <xacro:unless value="${joint_limited}">
@@ -185,6 +185,6 @@
         </geometry>
       </collision>
-      <xacro:cylinder_inertial radius="0.075" length="${-1*__kinematics['wrist_1']['x']}" mass="${forearm_mass}">
-        <origin xyz="${0.5*__kinematics['forearm']['x']} 0.0 ${elbow_offset}" rpy="0 ${pi/2} 0" />
+      <xacro:cylinder_inertial radius="0.075" length="${-1*config_kinematics['wrist_1']['x']}" mass="${forearm_mass}">
+        <origin xyz="${0.5*config_kinematics['forearm']['x']} 0.0 ${elbow_offset}" rpy="0 ${pi/2} 0" />
       </xacro:cylinder_inertial>
     </link>
@@ -192,5 +192,5 @@
       <parent link="${prefix}forearm_link" />
       <child link = "${prefix}wrist_1_link" />
-      <origin xyz="${__kinematics['wrist_1']['x']} ${__kinematics['wrist_1']['y']} ${__kinematics['wrist_1']['z']}" rpy="${__kinematics['wrist_1']['roll']} ${__kinematics['wrist_1']['pitch']} ${__kinematics['wrist_1']['yaw']}" />
+      <origin xyz="${config_kinematics['wrist_1']['x']} ${config_kinematics['wrist_1']['y']} ${config_kinematics['wrist_1']['z']}" rpy="${config_kinematics['wrist_1']['roll']} ${config_kinematics['wrist_1']['pitch']} ${config_kinematics['wrist_1']['yaw']}" />
       <axis xyz="0 0 1" />
       <xacro:unless value="${joint_limited}">
@@ -224,5 +224,5 @@
         </geometry>
       </collision>
-      <xacro:cylinder_inertial radius="0.075" length="${-1*__kinematics['wrist_2']['y']}" mass="${wrist_1_mass}">
+      <xacro:cylinder_inertial radius="0.075" length="${-1*config_kinematics['wrist_2']['y']}" mass="${wrist_1_mass}">
         <origin xyz="0.0 0.0 0.0" rpy="0 0 0" />
       </xacro:cylinder_inertial>
@@ -231,5 +231,5 @@
       <parent link="${prefix}wrist_1_link" />
       <child link = "${prefix}wrist_2_link" />
-      <origin xyz="${__kinematics['wrist_2']['x']} ${__kinematics['wrist_2']['y']} ${__kinematics['wrist_2']['z']}" rpy="${__kinematics['wrist_2']['roll']} ${__kinematics['wrist_2']['pitch']} ${__kinematics['wrist_2']['yaw']}" />
+      <origin xyz="${config_kinematics['wrist_2']['x']} ${config_kinematics['wrist_2']['y']} ${config_kinematics['wrist_2']['z']}" rpy="${config_kinematics['wrist_2']['roll']} ${config_kinematics['wrist_2']['pitch']} ${config_kinematics['wrist_2']['yaw']}" />
       <axis xyz="0 0 1" />
       <xacro:unless value="${joint_limited}">
@@ -263,5 +263,5 @@
         </geometry>
       </collision>
-      <xacro:cylinder_inertial radius="0.075" length="${__kinematics['wrist_3']['y']}" mass="${wrist_2_mass}">
+      <xacro:cylinder_inertial radius="0.075" length="${config_kinematics['wrist_3']['y']}" mass="${wrist_2_mass}">
         <origin xyz="0.0 0.0 0.0" rpy="0 0 0" />
       </xacro:cylinder_inertial>
@@ -270,5 +270,5 @@
       <parent link="${prefix}wrist_2_link" />
       <child link = "${prefix}wrist_3_link" />
-      <origin xyz="${__kinematics['wrist_3']['x']} ${__kinematics['wrist_3']['y']} ${__kinematics['wrist_3']['z']}" rpy="${__kinematics['wrist_3']['roll']} ${__kinematics['wrist_3']['pitch']} ${__kinematics['wrist_3']['yaw']}" />
+      <origin xyz="${config_kinematics['wrist_3']['x']} ${config_kinematics['wrist_3']['y']} ${config_kinematics['wrist_3']['z']}" rpy="${config_kinematics['wrist_3']['roll']} ${config_kinematics['wrist_3']['pitch']} ${config_kinematics['wrist_3']['yaw']}" />
       <axis xyz="0 0 1" />
       <xacro:unless value="${joint_limited}">
